File: board.brd (EAGLE design)
At the start: 160 x 100 mm, 87 parts, among them IC1 LMZ10501SILT, IC2 TPS61088RHLR, Q1 IRFML8244TRPBF, Q2 IRFML8244TRPBF, Q3 IRFML8244TRPBF, Q4 IRFML8244TRPBF, Q5 IRFML8244TRPBF, U1 TB6612FNG, U3 STM32F405RG

Commit message: Voltmeter Monitors on Boost, Batt, Cell1 and 5V Power LED
Parts:
- added 5V_PWR: (no value), CASE-LED:CHIP-LED0603
- added C30, C35: 0.1u, CASE-RCL:C0603
- added C34: 10n, CASE-RCL:C0603
- added R22: 47k, CASE-RCL:R0603
- added R24, R27, R31: 10k, CASE-RCL:R0603
- added R25: 1k, CASE-RCL:R0603
- added R26, R28: 20k, CASE-RCL:R0603
- added R29, R30, R_MOSI, R_SCL, R_SCLK, R_SDA: 0, CASE-RCL:R0603
- added SW: SPDT-500SSP1S1M6QEA, Isaks Bibliotek:500SSP1S1M6QEA
- added U$6, U$7: SPLITTER, Isaks Bibliotek:SPLITTER
- added U2: MPU6500, Isaks Bibliotek:QFN40P300X300X95-25T154X170
- added X1: JST-XH, JST XH Connectors:JST-XH-03-PACKAGE-LONG-PAD
- moved C19 905.5 mm to (-214.6, 20.3)
- moved C26 905.5 mm to (-224.8, -11.4)
- moved R18 905.5 mm to (-215.9, 52.1)
- moved C14 905.5 mm to (-207.0, 106.7)
- moved C15 905.5 mm to (-207.0, 101.6)
- moved C16 905.5 mm to (-214.6, 95.2)
- moved C17 905.5 mm to (-214.6, 88.9)
- moved C18 905.5 mm to (-215.9, 82.5)
- moved C20 905.5 mm to (-214.6, 14.0)
- moved C21 905.5 mm to (-215.9, 36.8)
- moved C22 905.5 mm to (-214.6, 7.62)
- moved C23 905.5 mm to (-215.9, 31.8)
- moved C24 905.5 mm to (-214.6, 1.27)
- moved C25 905.5 mm to (-214.6, -5.08)
- moved C27 905.5 mm to (-224.8, -16.5)
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Connections:
- new net !CS: R30.1
- new net INT: U2.12
- new net MISO: U2.9
- new net MOSI: R_MOSI.1
- new net N$28: C30.1, U2.10
- new net N$29: R_MOSI.2, R_SDA.2, U2.24
- new net N$30: R_SCL.2, R_SCLK.2, U2.23
- new net N$31: 5V_PWR.C, R25.2
- new net N$33: R26.2, X1.2
- new net N$36: R29.2, R30.2, U2.22
- new net N$38: R28.2, SW.2_COM, SW.3, X1.3
- new net SCL: R_SCL.1
- new net SCLK: R_SCLK.1
- new net SDA: R_SDA.1
- new net VOLM_BATT: R28.1, R31.2
- new net VOLM_CELL1: R26.1, R27.2
- new net VOLTM_BOOST: R22.1, R24.2
- net 12V: now also R22.2
- net 3.3VA: now also C34.1, C35.1, R29.1, U2.13, U2.8
- net 5V: now also 5V_PWR.A
- net GND: now also R27.1, R31.1, U$6.2, U$7.2, X1.1
- net GND_A: now also C30.2, C34.2, C35.2, U2.11, U2.18, U2.20
- net GND_M: now also U$6.1
- net GND_SW: now also R24.1, U$7.1
- net N$26: now also R25.1
- net V_BAT: now also SW.1
