File: board.sch (EAGLE design)
At the start: 130 parts, among them IC1 LMZ10501SILT, IC2 TPS61088RHLR, Q1 IRFML8244TRPBF, Q2 IRFML8244TRPBF, Q3 IRFML8244TRPBF, Q4 IRFML8244TRPBF, Q5 IRFML8244TRPBF, U1 TB6612FNG, U3 STM32F405RG, U4 BMI088, X1 JST-XH

Commit message: Eagle 9.5 persistent group update
Parts:
- removed D1, D2, D3, D7: SFH_4545, Isaks Bibliotek:SFH_4545
- removed IC1: LMZ10501SILT, Isaks Bibliotek:LMZ10501SILT
- added FL_EMITTER, FR_EMITTER, L_EMITTER, R_EMITTER: SFH_4545, Isaks Bibliotek:SFH_4545
- added IC3: LMZ10501, Isaks Bibliotek:LMZ10501
Connections:
- removed net N$28: U3.PB11, U3.PC13-TAMPER-RTC, U3.PC14-OSC32_IN, U3.PC15-OSC32_OUT, U3.PH0_OSC_IN, U3.PH1_OSC_OUT
- removed net N$29: U3.PA12, U3.PC12, U3.PC6, U3.PC7, U3.PC8
- removed net N$30: BTN_RST.1, BTN_RST.2, C36.2
- net 2V: now also FL_EMITTER.+_ANODE, FR_EMITTER.+_ANODE, IC3.FB, IC3.VOUT, L_EMITTER.+_ANODE, R_EMITTER.+_ANODE; no longer D1.+_ANODE, D2.+_ANODE, D3.+_ANODE, D7.+_ANODE, IC1.FB, IC1.VOUT
- net 5V: now also HC-05.VIN, IC3.VIN; no longer HC-05.+5V, IC1.VIN
- net GND: now also BTN_RST.1, BTN_RST.2, C36.2, IC3.EP, IC3.PGND, IC3.SGND; no longer IC1.EP, IC1.PGND, IC1.SGND
- net HEADER_RX: now also DEBUG.5
- net HEADER_TX: now also DEBUG.7
- net N$10: now also IC3.VREF; no longer IC1.VREF
- net N$11: now also IC3.VCON; no longer IC1.VCON
- net N$12: now also R_EMITTER.-_CATHODE; no longer D7.-_CATHODE
- net N$14: now also FR_EMITTER.-_CATHODE; no longer D3.-_CATHODE
- net N$2: now also L_EMITTER.-_CATHODE; no longer D1.-_CATHODE
- net N$5: now also FL_EMITTER.-_CATHODE; no longer D2.-_CATHODE
- net RX: no longer DEBUG.5
- net TX: no longer DEBUG.7
Other:
- note added: "Driver: TB6612FND"
- note added: "Driver: TPS61088RHLR switch mode boost regulator"
- note added: "Emitter: SFH4545 IR Diode"
- note added: "Interface: SWD & UART Remeber to choose where RX and TX goes with SB01-04 (Solderbridge)"
- note added: "Jerry the micromouse, high performance micromouse Created by: Isak Åslund"
- note added: "Motor: Faulhaber 1717SR Encoder: Faulhaber IES-1024 Connector: IDC-6Pin - DIN41651"
- note added: "Reciever: TEFT4300 IR transistor"
- note added: "STM32F405RG"
- note added: "Sensor: Bosch - BMI088 3-axis Accelerometer + 3-axis Gyro"
- note removed: "Debug SWD + UART"
- note removed: "Emitter System SFH4545"
- note removed: "IMU Bosch - BMI088"
- note removed: "Microcontroller STM32F405RG"
- note removed: "Motor Connector IDC-6Pin - DIN41651"
- note removed: "Motor Driver TB6612FND Dual"
- note removed: "Motor Supply TPS61088 - 12V"
- note removed: "Receiver System TEFT4300"
- note removed: "User Interface"
- moved on the sheet: 5V_PWR, BTN_RST, BTN_SEL, C1, C10, C11, C12, C13, C14, C15, C16, C17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

Commit message: 3D Packages update
Parts:
- renumbered JP1 to BOOT_JUMPERS
Other:
- moved on the sheet: IC3
