File: hardware/pcb/board.brd (EAGLE design)
At the start: 80 x 100 mm, 135 parts, among them IC2 TPS61088RHLR, IC3 LMZ10501, Q1 IRFML8244TRPBF, Q2 IRFML8244TRPBF, Q3 IRFML8244TRPBF, Q4 IRFML8244TRPBF, Q5 IRFML8244TRPBF, U1 TB6612FNG, U3 STM32F405RG, U4 BMI088

Commit message: Folder structure update and routing on PCB
Routing:
- net GND: track 559.8 -> 613.8 mm, vias 18 -> 22
- net L_RECEIVER: track 144.3 -> 151.8 mm, vias 3 -> 4
- net N$5: track 21.5 -> 23.9 mm
- net 2V: track 218.2 -> 216.1 mm
- net 3.3V: track 286.4 -> 284.7 mm
- net N$14: track 30.1 -> 31.4 mm
- net BUZZER: track 99.2 -> 98.3 mm
- net N$4: track 6.77 -> 7.52 mm
- net MOTOR_R_1: track 9.99 -> 10.6 mm
- net MOTOR_L_1: track 20.9 -> 21.5 mm
- net 3.3VA: track 229.8 -> 229.2 mm
Other:
- board text added: "SELECT"
- board text added: "STM32F405RG"
- board text added: "TB6612FNG"
- board text removed: "JERRY"
