File: hardware/pcb/board.sch (EAGLE design)
At the start: 134 parts, among them IC2 TPS61088RHLR, IC3 LMZ10501, Q1 IRFML8244TRPBF, Q2 IRFML8244TRPBF, Q3 IRFML8244TRPBF, Q4 IRFML8244TRPBF, Q5 IRFML8244TRPBF, U1 TB6612FNG, U3 STM32F405RG, U4 BMI088

Commit message: Folder structure update and routing on PCB
Parts:
- added FP2: 10u, CASE-RCL:WE-CBF_0805
Connections:
- net GND: now also FP2.1
- net GND_A: now also FP2.2
Changed lines of the file:
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@@
 <setting verticaltext="up"/>
 </settings>
-<grid distance="1.27" unitdist="mm" unit="mm" style="lines" multiple="1" display="no" altdistance="0.01" altunitdist="inch" altunit="inch"/>
+<grid distance="0.1" unitdist="inch" unit="inch" style="lines" multiple="1" display="no" altdistance="0.01" altunitdist="inch" altunit="inch"/>
 <layers>
 <layer number="1" name="Top" color="4" fill="1" visible="no" active="no"/>
@@
 <part name="SUPPLY19" library="Isaks Bibliotek" library_urn="urn:adsk.eagle:library:11889733" deviceset="5V" device=""/>
 <part name="U$8" library="Isaks Bibliotek" library_urn="urn:adsk.eagle:library:11889733" deviceset="GND_A" device=""/>
-<part name="DEBUG" library="CASE-Pinhead" deviceset="PINHD-2X4" device="" package3d_urn="urn:adsk.eagle:package:22461/2"/>
+<part name="DEBUG" library="CASE-Pinhead" deviceset="PINHD-2X4" device="" package3d_urn="urn:adsk.eagle:package:22461/2" override_package3d_urn="urn:adsk.eagle:package:13090280/2" override_package_urn="urn:adsk.eagle:footprint:22351/1"/>
 <part name="SUPPLY16" library="Isaks Bibliotek" library_urn="urn:adsk.eagle:library:11889733" deviceset="3.3V" device=""/>
 <part name="GND28" library="Isaks Bibliotek" library_urn="urn:adsk.eagle:library:11889733" deviceset="GND" device=""/>
@@
 <part name="GND34" library="Isaks Bibliotek" library_urn="urn:adsk.eagle:library:11889733" deviceset="GND" device=""/>
 <part name="SUPPLY27" library="Isaks Bibliotek" library_urn="urn:adsk.eagle:library:11889733" deviceset="3.3V" device=""/>
-<part name="BOOT" library="CASE-Pinhead" deviceset="PINHD-2X3" device="" package3d_urn="urn:adsk.eagle:package:22462/2"/>
+<part name="BOOT" library="CASE-Pinhead" deviceset="PINHD-2X3" device="" package3d_urn="urn:adsk.eagle:package:22462/2" override_package3d_urn="urn:adsk.eagle:package:13090277/2" override_package_urn="urn:adsk.eagle:footprint:22348/1"/>
 <part name="SUPPLY29" library="SparkFun-PowerSymbols" deviceset="3.3V" device=""/>
 <part name="GND36" library="SparkFun-PowerSymbols" deviceset="GND" device=""/>
@@
 <part name="TP_5V" library="Isaks Bibliotek" library_urn="urn:adsk.eagle:library:11889733" deviceset="TEST-POINT" device="3X5"/>
 <part name="TP_12V" library="Isaks Bibliotek" library_urn="urn:adsk.eagle:library:11889733" deviceset="TEST-POINT" device="3X5"/>
+<part name="FP2" library="CASE-RCL" deviceset="WE-CBF_0805" device="" package3d_urn="urn:adsk.eagle:package:5332310/3" value="10u"/>
 </parts>
 <sheets>
@@
 <attribute name="NAME" x="219.71" y="457.2" size="1.778" layer="95" font="vector"/>
 </instance>
+<instance part="FP2" gate="G$1" x="114.3" y="264.16" smashed="yes" rot="R90">
+<attribute name="VALUE" x="113.03" y="267.97" size="1.778" layer="96" rot="R180"/>
+</instance>
 </instances>
 <busses>
@@
 <junction x="81.28" y="264.16" grouprefs="POWER_REGULATION"/>
 <pinref part="GND20" gate="1" pin="GND"/>
+<pinref part="FP2" gate="G$1" pin="1"/>
+<wire x1="106.68" y1="264.16" x2="101.6" y2="264.16" width="0.1524" layer="91"/>
+<junction x="101.6" y="264.16"/>
 </segment>
 <segment>
@@
 <junction x="132.08" y="264.16" grouprefs="POWER_REGULATION"/>
 <pinref part="U$3" gate="G$1" pin="GND_A"/>
+<pinref part="FP2" gate="G$1" pin="2"/>
+<wire x1="121.92" y1="264.16" x2="127" y2="264.16" width="0.1524" layer="91"/>
+<junction x="127" y="264.16"/>
 </segment>
 <segment>
@@
 will not be understood (or retained) with this version.
 </note>
+<note version="9.4" severity="warning">
+Since Version 9.4, EAGLE supports the overriding of 3D packages
+in schematics and board files. Those overridden 3d packages
+will not be understood (or retained) with this version.
+</note>

Commit message: TPS61088 update
Parts:
- C21: value 27p -> 15p
- C23: value 560p -> 330p
- R20: value 30k -> 56k
Changed lines of the file:
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@@
 <drawing>
 <settings>
-<setting alwaysvectorfont="no"/>
+<setting alwaysvectorfont="yes"/>
 <setting verticaltext="up"/>
 </settings>
@@
 <part name="R19" library="CASE-RCL" deviceset="R0603" device="" package3d_urn="urn:adsk.eagle:package:5332309/4" value="20k"/>
 <part name="GND18" library="Isaks Bibliotek" library_urn="urn:adsk.eagle:library:11889733" deviceset="GND_SW" device=""/>
-<part name="R20" library="CASE-RCL" deviceset="R0603" device="" package3d_urn="urn:adsk.eagle:package:5332309/4" value="30k"/>
-<part name="C21" library="CASE-RCL" deviceset="C0603" device="" package3d_urn="urn:adsk.eagle:package:5332305/5" value="27p"/>
-<part name="C23" library="CASE-RCL" deviceset="C0603" device="" package3d_urn="urn:adsk.eagle:package:5332305/5" value="560p"/>
+<part name="R20" library="CASE-RCL" deviceset="R0603" device="" package3d_urn="urn:adsk.eagle:package:5332309/4" value="56k"/>
+<part name="C21" library="CASE-RCL" deviceset="C0603" device="" package3d_urn="urn:adsk.eagle:package:5332305/5" value="15p"/>
+<part name="C23" library="CASE-RCL" deviceset="C0603" device="" package3d_urn="urn:adsk.eagle:package:5332305/5" value="330p"/>
 <part name="GND19" library="Isaks Bibliotek" library_urn="urn:adsk.eagle:library:11889733" deviceset="GND_SW" device=""/>
 <part name="R21" library="CASE-RCL" deviceset="R0603" device="" package3d_urn="urn:adsk.eagle:package:5332309/4" value="112k"/>
